Commit message: make both axes move freely

File: final-project/xycartpole.urdf (robot description, URDF)
Before this commit: robot physics, 5 links, 4 joints
Links:
- removed link parallelBar2
- added link gimbal
Joints:
- removed joint cart_to_pole
- removed joint slider_to_parallel2
- added joint cart_to_gimabl: type continuous, parent cart, child gimbal, origin xyz=0.0 0.0 0, axis 1 0 0
- added joint gimabl_to_pole: type continuous, parent gimbal, child pole, origin xyz=0.0 0.0 0, axis 0 1 0
- joint slider_to_parallel1: child parallelBar1 -> slideBar; parent slideBar -> parallelBar1
